File: SiPM_readout/SIPM_readout.sch (EAGLE design)
At the start: 23 parts, among them J1 350180, J2 350180, J3 350180, J4 350180, J5 350180, U1 AD8000YRDZ-REEL7, U2 AD8000YRDZ-REEL7, U3 AD8000YRDZ-REEL7

Commit message: MPPC
Parts:
- removed U2, U3: AD8000YRDZ-REEL7, SiPM_AD8000:AD8000YRDZ-REEL7
- added AMP2, AMP3: AD8000YRDZ-REEL7, SiPM_AD8000:AD8000YRDZ-REEL7
- added MPPC: SSW-101-02-G-D, con-samtec:SSW-101-02-G-D
- added R7, R8: 3266W-1-102LF, SiPM_Trim_resistor:3266W-1-102LF
- added R9: ESR03EZPF1001, SiPM_R11:ESR03EZPF1001
- renumbered J1 to VIN, J2 to GND, J3 to +FB, J4 to -FB, J5 to VOUT, U1 to AMP1
Connections:
- removed net N$13: U2.+IN, U3.+IN
- new net N$1: AMP1.OUTPUT, R8.3
- new net N$18: AMP2.OUTPUT, R9.1
- new net N$4: AMP1.-IN, R4.1, R7.2
- net +FB: now also AMP2.+VS, AMP3.+VS; no longer U2.+VS, U3.+VS
- net -FB: now also AMP2.-VS, AMP3.-VS; no longer U2.-VS, U3.-VS
- net GND: now also AMP2.+IN, AMP2.EPAD, AMP3.+IN, AMP3.EPAD, R7.1, R8.1; no longer U2.EPAD, U3.EPAD
- net N$10: now also AMP2.NC; no longer U2.NC
- net N$11: now also AMP2.FEEDBACK; no longer U2.FEEDBACK
- net N$12: now also AMP2.-IN; no longer U2.-IN
- net N$14: now also AMP3.!POWERDOWN; no longer U3.!POWERDOWN
- net N$15: now also AMP3.NC; no longer U3.NC
- net N$16: now also AMP3.FEEDBACK; no longer U3.FEEDBACK
- net N$17: now also AMP3.-IN, R9.2; no longer U3.-IN
- net N$2: now also MPPC-2.1
- net N$3: now also R7.3
- net N$8: now also R8.2; no longer AMP1.-IN, R4.1
- net N$9: now also AMP2.!POWERDOWN; no longer U2.!POWERDOWN
- net VIN: now also MPPC-1.1
- net VOUT: now also AMP3.OUTPUT
Other:
- moved on the sheet: C6, C7, C8, C9, R5, R6

Commit message: mppc
Parts:
- added GND1: 350180, SiPM_banana:350180
Connections:
- removed net N$8: R8.2
- net GND: now also GND1.1
- net N$12: now also R8.2
Changed lines of the file:
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@@
 <part name="R9" library="SiPM_R11" deviceset="ESR03EZPF1001" device=""/>
 <part name="MPPC" library="con-samtec" library_urn="urn:adsk.eagle:library:184" deviceset="SSW-101-02-G" device="-D"/>
+<part name="GND1" library="SiPM_banana" deviceset="350180" device=""/>
 </parts>
 <sheets>
@@
 <instance part="MPPC" gate="-2" x="91.44" y="40.64" smashed="yes" rot="R270">
 <attribute name="NAME" x="92.202" y="43.688" size="1.524" layer="95" rot="R90"/>
+</instance>
+<instance part="GND1" gate="G$1" x="45.72" y="58.42" smashed="yes">
+<attribute name="NAME" x="40.64" y="62.23" size="1.778" layer="95"/>
+<attribute name="VALUE" x="40.64" y="54.61" size="1.778" layer="96" align="top-left"/>
 </instance>
 </instances>
@@
 <pinref part="AMP3" gate="A" pin="+IN"/>
 </segment>
+<segment>
+<pinref part="GND1" gate="G$1" pin="1"/>
+<wire x1="35.56" y1="58.42" x2="33.02" y2="58.42" width="0.1524" layer="91"/>
+<label x="33.02" y="58.42" size="1.778" layer="95" rot="R180" xref="yes"/>
+</segment>
 </net>
 <net name="+FB" class="0">
@@
 <pinref part="AMP2" gate="A" pin="-IN"/>
 <pinref part="R5" gate="A" pin="1"/>
+<pinref part="R8" gate="A" pin="2"/>
+<wire x1="309.88" y1="22.86" x2="302.26" y2="22.86" width="0.1524" layer="91"/>
 </segment>
 </net>
@@
 </segment>
 </net>
-<net name="N$8" class="0">
-<segment>
-<pinref part="R8" gate="A" pin="2"/>
-<wire x1="302.26" y1="22.86" x2="307.34" y2="22.86" width="0.1524" layer="91"/>
-</segment>
-</net>

Commit message: 2nd
Parts:
- removed C3: 1210AC101KAT1A, SiPM_C5:1210AC101KAT1A
- removed C4, C5, C6, C7, C8, C9: C3225C0G1H104J250AA, SiPM_C6:C3225C0G1H104J250AA
- removed R7, R8: 3266W-1-102LF, SiPM_Trim_resistor:3266W-1-102LF
- added C10: CGA3E2C0G1H101J080AA, SiPM_100p:CGA3E2C0G1H101J080AA
- added C11, C12, C13, C14, C15, C16: CL10B104KB8NNNL, SiPM_01u:CL10B104KB8NNNL
- added R10, R11: 3214W-1-103E, SiPM_trim:3214W-1-103E
Connections:
- net +FB: now also C12.1, C14.1, C16.1; no longer C5.1, C7.1, C9.1
- net -FB: now also C11.1, C13.1, C15.1; no longer C4.1, C6.1, C8.1
- net GND: now also C11.2, C12.2, C13.2, C14.2, C15.2, C16.2, R10.1, R11.1; no longer C4.2, C5.2, C6.2, C7.2, C8.2, C9.2, R7.1, R8.1
- net N$1: now also R10.3; no longer R8.3
- net N$12: now also R10.2; no longer R8.2
- net N$2: now also C10.1; no longer C3.1
- net N$3: now also C10.2, R11.3; no longer C3.2, R7.3
- net N$4: now also R11.2; no longer R7.2
Other:
- moved on the sheet: AMP1, R4
