File: SiPM_readout/SIPM_readout.brd (EAGLE design)
At the start: 160 x 100 mm, 27 parts

Commit message: mppc
Parts:
- added GND1: 350180, SiPM_banana:TE_350180
- moved R9 135.4 mm to (48.6, 71.6)
- moved +FB 135.4 mm to (47.5, 86.1), turned to 90 degrees
- moved R8 125.7 mm to (38.4, 76.9), flipped to the bottom
- moved VOUT 121.9 mm to (56.0, 85.5)
- moved R7 120.0 mm to (33.9, 78.5), turned to 90 degrees
- moved C5 113.1 mm to (48.9, 82.7), turned to 180 degrees
- moved AMP2 110.5 mm to (45.4, 77.4), flipped to the bottom, turned to 90 degrees
- moved C7 107.7 mm to (44.4, 83.0), flipped to the bottom
- moved C9 103.1 mm to (40.9, 82.8)
- moved VIN 102.1 mm to (34.9, 85.6), turned to 90 degrees
- moved GND 102.0 mm to (35.0, 69.1), turned to 270 degrees
- moved MPPC 99.4 mm to (11.2, 78.1), turned to 180 degrees
- moved AMP3 92.4 mm to (50.5, 77.5), turned to 90 degrees
- moved R5 92.3 mm to (47.0, 73.0), flipped to the bottom, turned to 180 degrees
- moved -FB 91.9 mm to (47.4, 69.0), turned to 270 degrees
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Connections:
- removed net N$8: R8.2
- net GND: now also GND1.1
- net N$12: now also R8.2
Other:
- board size 160 x 100 mm -> 57 x 37.5 mm

Commit message: mppc
Parts:
- moved C1 12.9 mm to (31.6, 79.2)
- moved C2 12.0 mm to (35.1, 79.3)
- moved R2 7.13 mm to (22.6, 76.7), turned to 90 degrees
- moved R7 5.04 mm to (32.7, 73.6)
- moved R1 3.52 mm to (29.0, 79.0)
- moved +FB 3.45 mm to (44.1, 86.7)
- moved C6 2.77 mm to (55.0, 70.8), turned to 0 degrees
- moved VIN 1.71 mm to (33.3, 86.2)
- moved GND 1.70 mm to (36.6, 69.2)
- moved C3 1.39 mm to (17.6, 75.8)
- moved C5 1.08 mm to (48.2, 83.6)
- moved MPPC 1.03 mm to (11.7, 79.0)
- moved C8 1.00 mm to (42.0, 71.7), turned to 0 degrees
- moved R3 0.82 mm to (21.5, 75.1)
- moved C7 0.71 mm to (44.5, 83.7)
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Routing:
- net +FB: track 0.00 -> 30.7 mm
- net N$3: track 0.00 -> 14.0 mm
- net N$18: track 0.00 -> 12.6 mm, vias 0 -> 1
- net N$2: track 0.00 -> 11.8 mm
- net GND: track 0.00 -> 8.78 mm
- net -FB: track 0.00 -> 8.26 mm
- net N$4: track 0.00 -> 7.76 mm
- net VOUT: track 0.00 -> 7.49 mm
- net N$17: track 0.00 -> 3.46 mm
- net N$11: track 0.00 -> 1.91 mm
- net N$16: track 0.00 -> 1.89 mm
- net N$12: track 0.00 -> 1.81 mm
- net N$7: track 0.00 -> 1.78 mm
- added copper zone on layer 1, net -FB
- added copper zone on layer 1, net GND
- added copper zone on layer 1, net VIN

Commit message: 2nd
Parts:
- removed C3: 1210AC101KAT1A, SiPM_C5:CAP_1210_AVX
- removed C4, C5, C6, C7, C8, C9: C3225C0G1H104J250AA, SiPM_C6:CAP_3225_TDK
- removed R7, R8: 3266W-1-102LF, SiPM_Trim_resistor:POT_3266W
- added C10: CGA3E2C0G1H101J080AA, SiPM_100p:CAP_1608_TDK
- added C11, C12, C13, C14, C15, C16: CL10B104KB8NNNL, SiPM_01u:CAP_CL10_SAM
- added R10, R11: 3214W-1-103E, SiPM_trim:POT_3214W
- moved AMP2 6.40 mm to (51.8, 77.2), flipped to the top
- moved R6 6.09 mm to (50.6, 78.9), flipped to the bottom
- moved R9 6.01 mm to (50.5, 77.3), flipped to the bottom
- moved AMP3 5.75 mm to (49.2, 83.1), flipped to the bottom
- moved R5 3.41 mm to (50.5, 72.8), flipped to the top
- moved -FB 2.01 mm to (49.4, 69.2)
Connections:
- net +FB: now also C12.1, C14.1, C16.1; no longer C5.1, C7.1, C9.1
- net -FB: now also C11.1, C13.1, C15.1; no longer C4.1, C6.1, C8.1
- net GND: now also C11.2, C12.2, C13.2, C14.2, C15.2, C16.2, R10.1, R11.1; no longer C4.2, C5.2, C6.2, C7.2, C8.2, C9.2, R7.1, R8.1
- net N$1: now also R10.3; no longer R8.3
- net N$12: now also R10.2; no longer R8.2
- net N$2: now also C10.1; no longer C3.1
- net N$3: now also C10.2, R11.3; no longer C3.2, R7.3
- net N$4: now also R11.2; no longer R7.2
Routing:
- net +FB: track 30.7 -> 18.6 mm
- net N$12: track 1.81 -> 8.91 mm
- net N$1: track 0.00 -> 5.80 mm
- net N$18: track 12.6 -> 6.79 mm
- net GND: track 8.78 -> 4.50 mm
- net N$3: track 14.0 -> 10.6 mm
- net N$2: track 11.8 -> 8.93 mm
- net VOUT: track 7.49 -> 9.98 mm
- net -FB: track 8.26 -> 5.84 mm
- net N$16: track 1.89 -> 0.00 mm
- net N$4: track 7.76 -> 8.87 mm
- added copper zone on layer 16, net -FB
- added copper zone on layer 16, net GND

Commit message: compact
Parts:
- moved C16 54.8 mm to (47.5, 81.6), flipped to the bottom, turned to 180 degrees
- moved C15 51.3 mm to (53.2, 73.2)
- moved C14 46.7 mm to (49.8, 82.4), turned to 90 degrees
- moved C12 35.7 mm to (38.9, 83.1), turned to 90 degrees
- moved C11 18.1 mm to (41.4, 72.4), turned to 270 degrees
- moved C13 7.92 mm to (42.4, 73.0), turned to 0 degrees
- moved R6 7.12 mm to (46.5, 73.1)
- moved AMP3 6.96 mm to (45.2, 77.4)
- moved R9 6.78 mm to (46.5, 71.8)
- moved R2 2.97 mm to (25.6, 77.1), turned to 0 degrees
- moved C2 1.70 mm to (33.4, 79.2)
- moved C1 1.50 mm to (30.1, 79.2)
- moved AMP2 1.43 mm to (50.4, 77.5)
- moved R5 1.43 mm to (49.1, 73.3)
- moved C10 1.38 mm to (19.8, 77.0), turned to 270 degrees
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Routing:
- net -FB: track 5.84 -> 28.4 mm
- net N$18: track 6.79 -> 15.5 mm
- net N$2: track 8.93 -> 14.1 mm
- net VOUT: track 9.98 -> 14.4 mm
- net +FB: track 18.6 -> 23.0 mm, vias 0 -> 1
- net GND: track 4.50 -> 0.34 mm
- net N$3: track 10.6 -> 12.4 mm
- net N$16: track 0.00 -> 1.63 mm
- removed copper zone on layer 1, net -FB
- removed copper zone on layer 16, net -FB
