File: dc2dc6_new/PI3523/PI3523_EVAL_v2.brd (EAGLE design)
At the start: 70 x 80 mm, 43 parts

Commit message: test
Parts:
- moved R2 3.50 mm to (34.9, 48.1)
- moved R1 2.97 mm to (34.0, 45.8), turned to 0 degrees
- moved C5 1.60 mm to (33.1, 48.2), turned to 90 degrees
- moved R4 1.41 mm to (34.6, 16.1)
- moved R3 1.28 mm to (33.8, 13.7), turned to 0 degrees
- moved C6 0.20 mm to (33.0, 16.3)
Routing:
- net SGND: track 15.7 -> 28.8 mm
- net SGND2: track 14.4 -> 27.5 mm
- net EAIN: track 0.00 -> 7.72 mm, vias 0 -> 1
- net EAIN2: track 0.00 -> 7.18 mm, vias 0 -> 1
- net VOUT: track 40.5 -> 42.5 mm
- net COMP: track 0.00 -> 1.61 mm
- net N$3: track 0.00 -> 1.61 mm
- net R21_1: track 0.00 -> 1.53 mm
- net COMP2: track 0.00 -> 1.51 mm

Commit message: mppc
Routing:
- net PGND: track 123.0 -> 137.9 mm
- net VIN: track 70.2 -> 73.0 mm
Changed lines of the file:
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@@
 <contactref element="VIN" pad="1"/>
 <polygon width="0.1" layer="1">
-<vertex x="22" y="8.7"/>
-<vertex x="25" y="8.7"/>
+<vertex x="22" y="8.9"/>
+<vertex x="25" y="8.9"/>
 <vertex x="25" y="80"/>
 <vertex x="22" y="80"/>
@@
 <vertex x="-1" y="61.5"/>
 <vertex x="22" y="61.5"/>
-<vertex x="22" y="8.7"/>
-<vertex x="25" y="8.7"/>
+<vertex x="22" y="8.9"/>
+<vertex x="25" y="8.9"/>
 </polygon>
 <polygon width="0.1" layer="2">
@@
 <contactref element="U$2" pad="VIN28"/>
 <contactref element="U$2" pad="VIN29"/>
+<wire x1="22.5" y1="41.2" x2="22.5" y2="40.1" width="0.5" layer="1"/>
+<wire x1="23.5" y1="41.2" x2="23.5" y2="40.5" width="0.5" layer="1"/>
+<wire x1="23.5" y1="40.5" x2="23.4" y2="40.4" width="0.5" layer="1"/>
+<wire x1="24.5" y1="41.2" x2="24.5" y2="40.3" width="0.5" layer="1"/>
 </signal>
 <signal name="SGND">
@@
 <contactref element="U$2" pad="SYNC1"/>
 <contactref element="U$2" pad="VSP"/>
-<wire x1="30.5" y1="46.2" x2="29.5" y2="46.2" width="0.55" layer="1"/>
+<wire x1="30.5" y1="46.2" x2="30" y2="46.2" width="0.55" layer="1"/>
+<wire x1="30" y1="46.2" x2="29.5" y2="46.2" width="0.55" layer="1"/>
 <wire x1="29.5" y1="46.2" x2="29.5" y2="47.2" width="0.55" layer="1"/>
-<wire x1="29.5" y1="47.2" x2="29.5" y2="49.2" width="0.55" layer="1"/>
+<wire x1="29.5" y1="47.2" x2="29.5" y2="47.7" width="0.55" layer="1"/>
+<wire x1="29.5" y1="47.7" x2="29.5" y2="48.7" width="0.55" layer="1"/>
+<wire x1="29.5" y1="48.7" x2="29.5" y2="49.2" width="0.55" layer="1"/>
 <wire x1="29.5" y1="48.2" x2="29.5" y2="48.3" width="0.55" layer="1"/>
 <wire x1="31.5" y1="47.2" x2="31.5" y2="46.2" width="0.55" layer="1"/>
@@
 <vertex x="36" y="50.6"/>
 </polygon>
+<wire x1="26.5" y1="46.2" x2="26.5" y2="45.2" width="0.5" layer="1"/>
+<wire x1="26.5" y1="46.2" x2="28.5" y2="46.2" width="0.5" layer="1"/>
+<wire x1="28.5" y1="46.2" x2="28.5" y2="47.1" width="0.5" layer="1"/>
+<wire x1="28.5" y1="47.1" x2="28.5" y2="48.2" width="0.5" layer="1"/>
+<wire x1="28.5" y1="48.2" x2="27.5" y2="48.2" width="0.5" layer="1"/>
+<wire x1="27.5" y1="48.2" x2="26.5" y2="48.2" width="0.5" layer="1"/>
+<wire x1="26.5" y1="48.2" x2="26.5" y2="46.2" width="0.5" layer="1"/>
+<wire x1="27.5" y1="46.2" x2="27.5" y2="48.2" width="0.5" layer="1"/>
+<wire x1="26.5" y1="47.2" x2="28.4" y2="47.2" width="0.5" layer="1"/>
+<wire x1="28.4" y1="47.2" x2="28.5" y2="47.1" width="0.5" layer="1"/>
+<wire x1="20.5" y1="50.2" x2="20.5" y2="52" width="0.5" layer="1"/>
+<wire x1="20.5" y1="52" x2="20.6" y2="52.1" width="0.5" layer="1"/>
 </signal>
 <signal name="COMP">
@@
 <wire x1="26.5" y1="50.2" x2="26.5" y2="49.2" width="0.3" layer="1"/>
 <wire x1="26.5" y1="50.2" x2="26.4" y2="50.3" width="0.3" layer="1"/>
-<wire x1="26.5" y1="50.2" x2="26.5" y2="51.8" width="0.3" layer="1"/>
-<wire x1="26.5" y1="51.8" x2="26.8" y2="52.1" width="0.3" layer="1"/>
+<wire x1="26.7" y1="52" x2="26.8" y2="52.1" width="0.3" layer="1"/>
+<wire x1="26.5" y1="50.2" x2="26.5" y2="51.8" width="0.5" layer="1"/>
+<wire x1="26.5" y1="51.8" x2="26.7" y2="52" width="0.5" layer="1"/>
 </signal>
 <signal name="VS1">

Commit message: compact
Routing:
- net PGND: track 137.9 -> 324.7 mm
- net VIN: track 73.0 -> 177.8 mm
- net VOUT2: track 54.9 -> 106.8 mm
- net VOUT: track 42.5 -> 88.2 mm
- net VS12: track 0.00 -> 24.9 mm
- net VS1: track 0.28 -> 24.1 mm
