File: dc2dc6_new/PI3523/PI3523_EVAL_v2.brd (EAGLE design)
At the start: 70 x 80 mm, 43 parts

Commit message: HV
Other:
- board text added: "KOREA UNIV. Elementary Particle Physics Lab. Supported by SNU"
- board text removed: "KOREA UNIV. Elementary Particle Lab. Supported by SNU"
Changed lines of the file:
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@@
 <layers>
 <layer number="1" name="Top" color="4" fill="1" visible="yes" active="yes"/>
-<layer number="2" name="Route2" color="16" fill="1" visible="no" active="yes"/>
+<layer number="2" name="Route2" color="16" fill="1" visible="yes" active="yes"/>
 <layer number="3" name="Route3" color="17" fill="1" visible="no" active="no"/>
 <layer number="4" name="Route4" color="18" fill="1" visible="no" active="no"/>
@@
 <layer number="13" name="Route13" color="21" fill="1" visible="no" active="no"/>
 <layer number="14" name="Route14" color="22" fill="1" visible="no" active="no"/>
-<layer number="15" name="Route15" color="23" fill="1" visible="no" active="yes"/>
-<layer number="16" name="Bottom" color="1" fill="1" visible="no" active="yes"/>
+<layer number="15" name="Route15" color="23" fill="1" visible="yes" active="yes"/>
+<layer number="16" name="Bottom" color="1" fill="1" visible="yes" active="yes"/>
 <layer number="17" name="Pads" color="2" fill="1" visible="yes" active="yes"/>
 <layer number="18" name="Vias" color="2" fill="1" visible="yes" active="yes"/>
@@
 </layers>
 <board>
-<fusionsync huburn="a.cGVyc29uYWw6dWUyOWYzNGEwMQ" projecturn="a.cGVyc29uYWw6dWUyOWYzNGEwMSMyMDIxMDQwMTM5ODc3OTY4MQ" f3durn="urn:adsk.wipprod:dm.lineage:KhInf_MFSzO_OmyKsKN06A" pcbguid="" lastpulledtime="2021-04-05T08:38:54Z" lastsyncedchangeguid="" latestrevisionid="b34aaca9-b2b8-4449-8c79-9344c58de8cb" lastsyncedrevisionid="b34aaca9-b2b8-4449-8c79-9344c58de8cb" lastboardhashguid="192832a3-b05f-bed8-089c-32f4dcce668d" lastpushedtime="2021-06-17T02:46:32Z" linktopcb3d="true"/>
+<fusionsync huburn="a.cGVyc29uYWw6dWUyOWYzNGEwMQ" projecturn="a.cGVyc29uYWw6dWUyOWYzNGEwMSMyMDIxMDQwMTM5ODc3OTY4MQ" f3durn="urn:adsk.wipprod:dm.lineage:KhInf_MFSzO_OmyKsKN06A" pcbguid="" lastpulledtime="2021-04-05T08:38:54Z" lastsyncedchangeguid="" latestrevisionid="b34aaca9-b2b8-4449-8c79-9344c58de8cb" lastsyncedrevisionid="b34aaca9-b2b8-4449-8c79-9344c58de8cb" lastboardhashguid="192832a3-b05f-bed8-089c-32f4dcce668d" lastpushedtime="2021-06-17T02:46:32Z" linktopcb3d="false"/>
 <plain>
 <rectangle x1="0" y1="0" x2="180" y2="150" layer="108"/>
@@
 <wire x1="60.44625" y1="14.4425" x2="60.64625" y2="14.3845" width="0.1" layer="25"/>
 <text x="67" y="6" size="1" layer="25" font="vector" rot="R180">KOREA UNIV.
-Elementary Particle Lab.
+Elementary Particle Physics Lab.
 Supported by SNU</text>
 <text x="37.5" y="75" size="1.3" layer="25" font="vector">DC to DC converter Ver. 6.1
