File: SiPM_readout_compact/SIPM_readout.sch (EAGLE design)
At the start: 26 parts

Commit message: c1c2
Parts:
- C1: value CGA6P3X7R1H335K250AB -> C3225X7S2A335M200ABCAP_3225_TDK-M; device SiPM_C3:CGA6P3X7R1H335K250AB -> SiPM_3.3uF:C3225X7S2A335M200ABCAP_3225_TDK-M
- C2: value C3225X7R1H105K160AA -> C3225X7R2A105K200AACAP_3225_TDK-M; device SiPM_C4:C3225X7R1H105K160AA -> SiPM_1uF:C3225X7R2A105K200AACAP_3225_TDK-M
Changed lines of the file:
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@@
 </groups>
 <parts>
-<part name="C1" library="SiPM_C3" deviceset="CGA6P3X7R1H335K250AB" device=""/>
-<part name="C2" library="SiPM_C4" deviceset="C3225X7R1H105K160AA" device=""/>
 <part name="R1" library="SiPM_R6" deviceset="RC0603FR-072ML" device=""/>
 <part name="R2" library="SiPM_R7" deviceset="RT0603BRD0710RL" device=""/>
@@
 <part name="VIN" library="con-molex" library_urn="urn:adsk.eagle:library:165" deviceset="22-23-2021" device="" package3d_urn="urn:adsk.eagle:package:8078633/1"/>
 <part name="VOUT" library="con-molex" library_urn="urn:adsk.eagle:library:165" deviceset="22-23-2021" device="" package3d_urn="urn:adsk.eagle:package:8078633/1"/>
+<part name="C1" library="SiPM_3.3uF" deviceset="C3225X7S2A335M200AB" device="CAP_3225_TDK-M"/>
+<part name="C2" library="SiPM_1uF" deviceset="C3225X7R2A105K200AA" device="CAP_3225_TDK-M"/>
 </parts>
 <sheets>
@@
 </plain>
 <instances>
-<instance part="C1" gate="A" x="20.32" y="35.56" smashed="yes" rot="R270">
-<attribute name="NAME" x="22.4028" y="39.6494" size="3.4798" layer="95" ratio="10" rot="SR270"/>
-</instance>
-<instance part="C2" gate="A" x="30.48" y="25.4" smashed="yes" rot="R270">
-<attribute name="NAME" x="32.5628" y="29.4894" size="3.4798" layer="95" ratio="10" rot="SR270"/>
-</instance>
 <instance part="R1" gate="A" x="40.64" y="25.4" smashed="yes" rot="R270">
 <attribute name="NAME" x="42.7228" y="27.5844" size="3.4798" layer="95" ratio="10" rot="SR270"/>
 </instance>
 <instance part="R2" gate="A" x="71.12" y="5.08" smashed="yes">
-<attribute name="VALUE" x="68.5038" y="-0.4572" size="3.4798" layer="96" ratio="10" rot="SR0"/>
 <attribute name="NAME" x="68.9356" y="7.1628" size="3.4798" layer="95" ratio="10" rot="SR0"/>
 </instance>
@@
 <instance part="R10" gate="A" x="294.64" y="33.02" smashed="yes" rot="R270">
 <attribute name="NAME" x="289.7124" y="30.1244" size="3.4798" layer="95" ratio="10" rot="SR270"/>
-<attribute name="VALUE" x="286.5628" y="31.1912" size="3.4798" layer="96" ratio="10" rot="SR270"/>
 </instance>
 <instance part="R11" gate="A" x="144.78" y="43.18" smashed="yes" rot="R270">
 <attribute name="NAME" x="139.8524" y="40.2844" size="3.4798" layer="95" ratio="10" rot="SR270"/>
-<attribute name="VALUE" x="136.7028" y="41.3512" size="3.4798" layer="96" ratio="10" rot="SR270"/>
 </instance>
 <instance part="C10" gate="A" x="119.38" y="20.32" smashed="yes">
-<attribute name="VALUE" x="114.2238" y="14.7828" size="3.4798" layer="96" ratio="10" rot="SR0"/>
 <attribute name="NAME" x="115.2906" y="22.4028" size="3.4798" layer="95" ratio="10" rot="SR0"/>
 </instance>
 <instance part="C11" gate="A" x="203.2" y="-2.54" smashed="yes">
-<attribute name="VALUE" x="198.0438" y="-8.0772" size="3.4798" layer="96" ratio="10" rot="SR0"/>
 <attribute name="NAME" x="199.1106" y="-0.4572" size="3.4798" layer="95" ratio="10" rot="SR0"/>
 </instance>
 <instance part="C12" gate="A" x="274.32" y="35.56" smashed="yes">
-<attribute name="VALUE" x="269.1638" y="30.0228" size="3.4798" layer="96" ratio="10" rot="SR0"/>
 <attribute name="NAME" x="270.2306" y="37.6428" size="3.4798" layer="95" ratio="10" rot="SR0"/>
 </instance>
 <instance part="C13" gate="A" x="330.2" y="-2.54" smashed="yes">
-<attribute name="VALUE" x="325.0438" y="-8.0772" size="3.4798" layer="96" ratio="10" rot="SR0"/>
 <attribute name="NAME" x="326.1106" y="-0.4572" size="3.4798" layer="95" ratio="10" rot="SR0"/>
 </instance>
 <instance part="C14" gate="A" x="401.32" y="35.56" smashed="yes">
-<attribute name="VALUE" x="396.1638" y="30.0228" size="3.4798" layer="96" ratio="10" rot="SR0"/>
 <attribute name="NAME" x="397.2306" y="37.6428" size="3.4798" layer="95" ratio="10" rot="SR0"/>
 </instance>
 <instance part="C15" gate="A" x="457.2" y="-2.54" smashed="yes">
-<attribute name="VALUE" x="452.0438" y="-8.0772" size="3.4798" layer="96" ratio="10" rot="SR0"/>
 <attribute name="NAME" x="453.1106" y="-0.4572" size="3.4798" layer="95" ratio="10" rot="SR0"/>
 </instance>
 <instance part="C16" gate="A" x="528.32" y="35.56" smashed="yes">
-<attribute name="VALUE" x="523.1638" y="30.0228" size="3.4798" layer="96" ratio="10" rot="SR0"/>
 <attribute name="NAME" x="524.2306" y="37.6428" size="3.4798" layer="95" ratio="10" rot="SR0"/>
 </instance>
@@
 <instance part="VOUT" gate="-2" x="96.52" y="93.98" smashed="yes">
 <attribute name="NAME" x="99.06" y="93.218" size="1.524" layer="95"/>
+</instance>
+<instance part="C1" gate="A" x="20.32" y="35.56" smashed="yes" rot="R270">
+<attribute name="NAME" x="22.4028" y="42.1894" size="3.4798" layer="95" ratio="10" rot="SR270"/>
+</instance>
+<instance part="C2" gate="A" x="30.48" y="25.4" smashed="yes" rot="R270">
+<attribute name="NAME" x="32.5628" y="29.4894" size="3.4798" layer="95" ratio="10" rot="SR270"/>
 </instance>
 </instances>
@@
 <label x="12.7" y="38.1" size="1.778" layer="95" rot="R180" xref="yes"/>
 <wire x1="12.7" y1="38.1" x2="20.32" y2="38.1" width="0.1524" layer="91"/>
-<pinref part="C1" gate="A" pin="1"/>
 <wire x1="20.32" y1="38.1" x2="20.32" y2="35.56" width="0.1524" layer="91"/>
 <wire x1="20.32" y1="38.1" x2="35.56" y2="38.1" width="0.1524" layer="91"/>
@@
 <wire x1="35.56" y1="38.1" x2="35.56" y2="30.48" width="0.1524" layer="91"/>
 <wire x1="35.56" y1="30.48" x2="30.48" y2="30.48" width="0.1524" layer="91"/>
-<pinref part="C2" gate="A" pin="1"/>
 <wire x1="30.48" y1="30.48" x2="30.48" y2="25.4" width="0.1524" layer="91"/>
 <wire x1="35.56" y1="30.48" x2="40.64" y2="30.48" width="0.1524" layer="91"/>
@@
 <junction x="35.56" y="38.1"/>
 <pinref part="MPPC" gate="-1" pin="1"/>
+<pinref part="C1" gate="A" pin="1"/>
+<pinref part="C2" gate="A" pin="1"/>
 </segment>
 <segment>
@@
 </segment>
 <segment>
-<pinref part="C1" gate="A" pin="2"/>
 <wire x1="20.32" y1="27.94" x2="20.32" y2="25.4" width="0.1524" layer="91"/>
 <label x="20.32" y="25.4" size="1.778" layer="95" rot="R270" xref="yes"/>
-</segment>
-<segment>
-<pinref part="C2" gate="A" pin="2"/>
+<pinref part="C1" gate="A" pin="2"/>
+</segment>
+<segment>
 <wire x1="30.48" y1="17.78" x2="30.48" y2="10.16" width="0.1524" layer="91"/>
 <wire x1="30.48" y1="10.16" x2="35.56" y2="10.16" width="0.1524" layer="91"/>
@@
 <junction x="66.04" y="5.08"/>
 <label x="66.04" y="0" size="1.778" layer="95" rot="R270" xref="yes"/>
-</segment>
-<segment>
+<pinref part="C2" gate="A" pin="2"/>
+</segment>
+<segment>
