File: SiPM_readout_compact/SIPM_readout.brd (EAGLE design)
At the start: 51 x 25 mm, 26 parts

Commit message: test
Parts:
- moved MPPC 1.10 mm to (13.8, 79.2)
Routing:
- net N$2: track 13.3 -> 12.2 mm
- net GND: vias 0 -> 17
Other:
- board size 51 x 25 mm -> 50 x 25 mm

Commit message: c1c2
Parts:
- C1: value CGA6P3X7R1H335K250AB -> C3225X7S2A335M200ABCAP_3225_TDK-M; device SiPM_C3:CAP_3225_TDK -> SiPM_3.3uF:CAP_3225_TDK-M
- C2: value C3225X7R1H105K160AA -> C3225X7R2A105K200AACAP_3225_TDK-M; device SiPM_C4:CAP_3225_TDK -> SiPM_1uF:CAP_3225_TDK-M
- moved C2 0.12 mm to (33.5, 79.2)
- moved C1 0.09 mm to (30.2, 79.2)
Changed lines of the file:
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@@
 </groups>
 <elements>
-<element name="C1" library="SiPM_C3" package="CAP_3225_TDK" value="CGA6P3X7R1H335K250AB" x="30.11" y="79.17" smashed="yes" rot="R270">
-<attribute name="BUILT_BY" value="EMA_UL_Team" x="-9.26" y="44.88" size="1.778" layer="27" rot="R270" display="off"/>
-<attribute name="MANUFACTURER_PART_NUMBER" value="CGA6P3X7R1H335K250AB" x="-9.26" y="44.88" size="1.778" layer="27" rot="R270" display="off"/>
-<attribute name="NAME" x="29.475" y="81.4466" size="1.27" layer="25" ratio="6" rot="SR90"/>
-<attribute name="SOURCELIBRARY" value="TDK_2015_05_22" x="-9.26" y="44.88" size="1.778" layer="27" rot="R270" display="off"/>
-<attribute name="VENDOR" value="TDK" x="-9.26" y="44.88" size="1.778" layer="27" rot="R270" display="off"/>
-</element>
-<element name="C2" library="SiPM_C4" package="CAP_3225_TDK" value="C3225X7R1H105K160AA" x="33.38" y="79.17" smashed="yes" rot="R270">
-<attribute name="BUILT_BY" value="EMA_UL_Team" x="-5.99" y="20.75" size="1.778" layer="27" rot="R270" display="off"/>
-<attribute name="MANUFACTURER_PART_NUMBER" value="C3225X7R1H105K160AA" x="-5.99" y="20.75" size="1.778" layer="27" rot="R270" display="off"/>
-<attribute name="NAME" x="32.5534" y="81.445" size="1.27" layer="25" ratio="6" rot="SR90"/>
-<attribute name="SOURCELIBRARY" value="TDK_2015_05_22" x="-5.99" y="20.75" size="1.778" layer="27" rot="R270" display="off"/>
-<attribute name="VENDOR" value="TDK" x="-5.99" y="20.75" size="1.778" layer="27" rot="R270" display="off"/>
-</element>
 <element name="R1" library="SiPM_R6" package="RC0603N_YAG" value="RC0603FR-072ML" x="27.8" y="79.2" smashed="yes" rot="R90">
 <attribute name="BUILT_BY" value="EMA_UL_Team" x="86.22" y="126.19" size="1.778" layer="27" rot="R90" display="off"/>
@@
 <attribute name="VALUE" x="51.44" y="80.06" size="1.016" layer="27" ratio="10" rot="R270"/>
 </element>
+<element name="C1" library="SiPM_3.3uF" package="CAP_3225_TDK-M" value="C3225X7S2A335M200ABCAP_3225_TDK-M" x="30.2" y="79.2" smashed="yes" rot="R270">
+<attribute name="BUILT_BY" value="EMA_UL_Team" x="30.2" y="79.2" size="1.778" layer="27" rot="R270" display="off"/>
+<attribute name="MANUFACTURER_PART_NUMBER" value="C3225X7S2A335M200AB" x="30.2" y="79.2" size="1.778" layer="27" rot="R270" display="off"/>
+<attribute name="NAME" x="28.965" y="84.0766" size="1.27" layer="25" ratio="6" rot="SR0"/>
+<attribute name="SOURCELIBRARY" value="TDK_2015_05_22" x="30.2" y="79.2" size="1.778" layer="27" rot="R270" display="off"/>
+<attribute name="VALUE" x="29.565" y="80.9272" size="1.27" layer="27" ratio="6" rot="SR270"/>
+<attribute name="VENDOR" value="TDK" x="30.2" y="79.2" size="1.778" layer="27" rot="R270" display="off"/>
+</element>
+<element name="C2" library="SiPM_1uF" package="CAP_3225_TDK-M" value="C3225X7R2A105K200AACAP_3225_TDK-M" x="33.5" y="79.2" smashed="yes" rot="R270">
+<attribute name="BUILT_BY" value="EMA_UL_Team" x="33.5" y="79.2" size="1.778" layer="27" rot="R270" display="off"/>
+<attribute name="MANUFACTURER_PART_NUMBER" value="C3225X7R2A105K200AA" x="33.5" y="79.2" size="1.778" layer="27" rot="R270" display="off"/>
+<attribute name="NAME" x="32.165" y="84.0766" size="1.27" layer="25" ratio="6" rot="SR0"/>
+<attribute name="SOURCELIBRARY" value="TDK_2015_05_22" x="33.5" y="79.2" size="1.778" layer="27" rot="R270" display="off"/>
+<attribute name="VALUE" x="32.865" y="80.9272" size="1.27" layer="27" ratio="6" rot="SR270"/>
+<attribute name="VENDOR" value="TDK" x="33.5" y="79.2" size="1.778" layer="27" rot="R270" display="off"/>
+</element>
 </elements>
 <signals>
 <signal name="VIN">
-<contactref element="C1" pad="1"/>
-<contactref element="C2" pad="1"/>
 <contactref element="R1" pad="2"/>
 <contactref element="MPPC" pad="1"/>
@@
 <via x="34.4" y="83.5" extent="1-16" drill="0.35"/>
 <via x="35.9" y="83.5" extent="1-16" drill="0.35" diameter="0.55"/>
+<contactref element="C1" pad="1"/>
+<contactref element="C2" pad="1"/>
 </signal>
 <signal name="GND">
@@
 <contactref element="AMP2" pad="EPAD"/>
 <contactref element="AMP3" pad="EPAD"/>
-<contactref element="C1" pad="2"/>
-<contactref element="C2" pad="2"/>
 <contactref element="R1" pad="1"/>
 <contactref element="R2" pad="2"/>
@@
 <via x="47" y="86.6" extent="1-16" drill="0.35"/>
 <via x="38.4" y="83.6" extent="1-16" drill="0.35"/>
+<contactref element="C1" pad="2"/>
+<contactref element="C2" pad="2"/>
 </signal>
 <signal name="+FB">

Commit message: HV
Other:
- board size 50 x 25 mm -> 50 x 24.9 mm
Changed lines of the file:
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@@
 <layer number="14" name="Route14" color="22" fill="1" visible="no" active="no"/>
 <layer number="15" name="Route15" color="23" fill="1" visible="no" active="no"/>
-<layer number="16" name="Bottom" color="1" fill="1" visible="yes" active="yes"/>
+<layer number="16" name="Bottom" color="1" fill="1" visible="no" active="yes"/>
 <layer number="17" name="Pads" color="2" fill="1" visible="yes" active="yes"/>
 <layer number="18" name="Vias" color="2" fill="1" visible="yes" active="yes"/>
@@
 <layer number="20" name="Dimension" color="24" fill="1" visible="yes" active="yes"/>
 <layer number="21" name="tPlace" color="7" fill="1" visible="yes" active="yes"/>
-<layer number="22" name="bPlace" color="7" fill="1" visible="yes" active="yes"/>
+<layer number="22" name="bPlace" color="7" fill="1" visible="no" active="yes"/>
 <layer number="23" name="tOrigins" color="15" fill="1" visible="yes" active="yes"/>
-<layer number="24" name="bOrigins" color="15" fill="1" visible="yes" active="yes"/>
+<layer number="24" name="bOrigins" color="15" fill="1" visible="no" active="yes"/>
 <layer number="25" name="tNames" color="7" fill="1" visible="yes" active="yes"/>
-<layer number="26" name="bNames" color="7" fill="1" visible="yes" active="yes"/>
+<layer number="26" name="bNames" color="7" fill="1" visible="no" active="yes"/>
 <layer number="27" name="tValues" color="7" fill="1" visible="no" active="yes"/>
 <layer number="28" name="bValues" color="7" fill="1" visible="no" active="yes"/>
@@
 <layer number="38" name="bTest" color="7" fill="1" visible="no" active="yes"/>
 <layer number="39" name="tKeepout" color="4" fill="11" visible="yes" active="yes"/>
-<layer number="40" name="bKeepout" color="1" fill="11" visible="yes" active="yes"/>
+<layer number="40" name="bKeepout" color="1" fill="11" visible="no" active="yes"/>
 <layer number="41" name="tRestrict" color="4" fill="10" visible="yes" active="yes"/>
-<layer number="42" name="bRestrict" color="1" fill="10" visible="yes" active="yes"/>
+<layer number="42" name="bRestrict" color="1" fill="10" visible="no" active="yes"/>
 <layer number="43" name="vRestrict" color="2" fill="10" visible="no" active="yes"/>
 <layer number="44" name="Drills" color="7" fill="1" visible="no" active="yes"/>
@@
 <layer number="50" name="dxf" color="7" fill="1" visible="no" active="no"/>
 <layer number="51" name="tDocu" color="7" fill="1" visible="yes" active="yes"/>
-<layer number="52" name="bDocu" color="7" fill="1" visible="yes" active="yes"/>
+<layer number="52" name="bDocu" color="7" fill="1" visible="no" active="yes"/>
 <layer number="53" name="tGND_GNDA" color="7" fill="1" visible="no" active="no"/>
 <layer number="54" name="bGND_GNDA" color="7" fill="1" visible="no" active="no"/>
@@
 <fusionsync huburn="a.cGVyc29uYWw6dWUyOWYzNGEwMQ" projecturn="a.cGVyc29uYWw6dWUyOWYzNGEwMSMyMDIxMDYxNjQyMDk2OTI1Ng" f3durn="urn:adsk.wipprod:dm.lineage:73l8zhv5RF-XBDXu35YORA" pcbguid="" lastpulledtime="" lastsyncedchangeguid="" latestrevisionid="a99baacc-6fba-49c1-9e69-8d64e022b22a" lastsyncedrevisionid="a99baacc-6fba-49c1-9e69-8d64e022b22a" lastboardhashguid="9c3b8375-83c7-0d3a-68b5-104893922fa0" lastpushedtime="2021-06-17T01:39:31Z" linktopcb3d="true"/>
 <plain>
-<wire x1="60.3" y1="64.8" x2="10.3" y2="64.7" width="0.1524" layer="20"/>
-<wire x1="10.3" y1="64.7" x2="10.3" y2="89.7" width="0.1524" layer="20"/>
+<wire x1="60.3" y1="64.8" x2="10.3" y2="64.8" width="0.1524" layer="20"/>
+<wire x1="10.3" y1="64.8" x2="10.3" y2="89.7" width="0.1524" layer="20"/>
 <wire x1="10.3" y1="89.7" x2="60.3" y2="89.7" width="0.1524" layer="20"/>
 <wire x1="60.3" y1="89.7" x2="60.3" y2="64.8" width="0.1524" layer="20"/>
@@
 <wire x1="15.86913125" y1="88.70725" x2="15.97313125" y2="88.67125" width="0.1" layer="25"/>
 <wire x1="15.97313125" y1="88.67125" x2="16.07313125" y2="88.64225" width="0.1" layer="25"/>
-<dimension x1="10.3" y1="89.7" x2="60.3" y2="89.7" x3="35.3" y3="94.3" textsize="1.778" layer="20"/>
 </plain>
 <attributes>
@@
 <contactref element="R10" pad="1"/>
 <polygon width="0.1" layer="16">
-<vertex x="11.4" y="65.5"/>
+<vertex x="10.3" y="65.5"/>
 <vertex x="60" y="65.5"/>
 <vertex x="60" y="89.69"/>
 <vertex x="37.4" y="89.69995625"/>
 <vertex x="37.4" y="79"/>
-<vertex x="11.4" y="79"/>
+<vertex x="10.3" y="79"/>
 </polygon>
 <contactref element="C11" pad="2"/>
